Commit message: some more find replaces for youbot_description to youbot-ros-pkg-kdl

File: robots/youbot.urdf (robot description, URDF)
Before this commit: robot youbot, 21 links, 20 joints
Links:
- link arm_link_0: geometry collision mesh filename=package://youbot-ros-pkg-kdl/meshes/youbot_arm/arm0_convex.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; visual mesh filename=package://youbot-ros-pkg-kdl/meshes/youbot_arm/arm0.dae
- link arm_link_1: geometry collision mesh filename=package://youbot-ros-pkg-kdl/meshes/youbot_arm/arm1_convex.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; visual mesh filename=package://youbot-ros-pkg-kdl/meshes/youbot_arm/arm1.dae
- link arm_link_2: geometry collision mesh filename=package://youbot-ros-pkg-kdl/meshes/youbot_arm/arm2_convex.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; visual mesh filename=package://youbot-ros-pkg-kdl/meshes/youbot_arm/arm2.dae
- link arm_link_3: geometry collision mesh filename=package://youbot-ros-pkg-kdl/meshes/youbot_arm/arm3_convex.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; visual mesh filename=package://youbot-ros-pkg-kdl/meshes/youbot_arm/arm3.dae
- link arm_link_4: geometry collision mesh filename=package://youbot-ros-pkg-kdl/meshes/youbot_arm/arm4_convex.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; visual mesh filename=package://youbot-ros-pkg-kdl/meshes/youbot_arm/arm4.dae
- link arm_link_5: geometry collision mesh filename=package://youbot-ros-pkg-kdl/meshes/youbot_arm/arm5_convex.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; visual mesh filename=package://youbot-ros-pkg-kdl/meshes/youbot_arm/arm5.dae
- link base_laser_front_link: geometry collision mesh filename=package://youbot-ros-pkg-kdl/meshes/sensors/hokuyo_convex.s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; visual mesh filename=package://youbot-ros-pkg-kdl/meshes/sensors/hokuyo.dae
- link base_link: geometry collision mesh filename=package://youbot-ros-pkg-kdl/meshes/youbot_base/base_convex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; visual mesh filename=package://youbot-ros-pkg-kdl/meshes/youbot_base/base.dae
- link gripper_finger_link_l: geometry collision mesh filename=package://youbot-ros-pkg-kdl/meshes/youbot_gripper/finger_c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; visual mesh filename=package://youbot-ros-pkg-kdl/meshes/youbot_gripper/finger.s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
- link gripper_finger_link_r: geometry collision mesh filename=package://youbot-ros-pkg-kdl/meshes/youbot_gripper/finger_c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; visual mesh filename=package://youbot-ros-pkg-kdl/meshes/youbot_gripper/finger.s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
- link gripper_palm_link: geometry collision mesh filename=package://youbot-ros-pkg-kdl/meshes/youbot_gripper/palm_con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; visual mesh filename=package://youbot-ros-pkg-kdl/meshes/youbot_gripper/palm.stl
- link plate_link: geometry collision mesh filename=package://youbot-ros-pkg-kdl/meshes/youbot_plate/plate_conv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; visual mesh filename=package://youbot-ros-pkg-kdl/meshes/youbot_plate/plate.dae

File: urdf/sensors/hokuyo_urg04_laser.urdf.xacro (robot description, xacro)
@@ -4,5 +4,5 @@
        xmlns:interface="http://playerstage.sourceforge.net/gazebo/xmlschema/#interface"
        xmlns:xacro="http://ros.org/wiki/xacro">
-  <include filename="$(find youbot_description)/urdf/sensors/hokuyo_urg04_laser.gazebo.xacro" />
+  <include filename="$(find youbot-ros-pkg-kdl)/urdf/sensors/hokuyo_urg04_laser.gazebo.xacro" />
   <xacro:macro name="hokuyo_urg04_laser" params="name parent *origin ros_topic update_rate min_angle max_angle">
     <joint name="${name}_hokuyo_urg04_laser_joint" type="fixed">
@@ -21,5 +21,5 @@
       	<origin xyz="0 0 0" rpy="0 0 0" />
 	<geometry>
-		<mesh filename="package://youbot_description/meshes/sensors/hokuyo.dae" />
+		<mesh filename="package://youbot-ros-pkg-kdl/meshes/sensors/hokuyo.dae" />
 	</geometry>
 	<material name="DarkGrey" />
@@ -28,5 +28,5 @@
 		<origin xyz="0 0 0" rpy="0 0 0" />
 		<geometry>
-			<mesh filename="package://youbot_description/meshes/sensors/hokuyo_convex.stl" />
+			<mesh filename="package://youbot-ros-pkg-kdl/meshes/sensors/hokuyo_convex.stl" />
 		</geometry>
 	</collision>

File: urdf/youbot_arm/arm.urdf.xacro (robot description, xacro)
@@ -4,7 +4,7 @@
         xmlns:interface="http://playerstage.sourceforge.net/gazebo/xmlschema/#interface"
         xmlns:xacro="http://ros.org/wiki/xacro">
-	<include filename="$(find youbot_description)/urdf/youbot_arm/arm.gazebo.xacro" />
-	<include filename="$(find youbot_description)/urdf/youbot_arm/arm.transmission.xacro" />
-        <include filename="$(find youbot_description)/urdf/youbot_arm/limits.urdf.xacro" />
+	<include filename="$(find youbot-ros-pkg-kdl)/urdf/youbot_arm/arm.gazebo.xacro" />
+	<include filename="$(find youbot-ros-pkg-kdl)/urdf/youbot_arm/arm.transmission.xacro" />
+        <include filename="$(find youbot-ros-pkg-kdl)/urdf/youbot_arm/limits.urdf.xacro" />
 	<xacro:macro name="youbot_arm" params="parent name *origin">
 		<!-- joint between base_link and arm_0_link -->
@@ -24,5 +24,5 @@
 				<origin xyz="0 0 0" rpy="0 0 0" />
 				<geometry>
-					<mesh filename="package://youbot_description/meshes/youbot_arm/arm0.dae" />
+					<mesh filename="package://youbot-ros-pkg-kdl/meshes/youbot_arm/arm0.dae" />
 				</geometry>
 				<material name="DarkGrey" />
@@ -32,5 +32,5 @@
 				<origin xyz="0 0 0" rpy="0 0 0"/>
 				<geometry>
-					<mesh filename="package://youbot_description/meshes/youbot_arm/arm0_convex.stl" />
+					<mesh filename="package://youbot-ros-pkg-kdl/meshes/youbot_arm/arm0_convex.stl" />
 					<!--<cylinder length="0.078" radius="0.093"/>-->
 				</geometry>
@@ -58,5 +58,5 @@
 				<origin xyz="0 0 0" rpy="0 0 0" />
 				<geometry>
-					<mesh filename="package://youbot_description/meshes/youbot_arm/arm1.dae" />
+					<mesh filename="package://youbot-ros-pkg-kdl/meshes/youbot_arm/arm1.dae" />
 				</geometry>
 				<!--<material name="Orange" />-->
@@ -66,5 +66,5 @@
 				<origin xyz="0 0 0" rpy="0 0 0" />
 				<geometry>
-					<mesh filename="package://youbot_description/meshes/youbot_arm/arm1_convex.stl" />
+					<mesh filename="package://youbot-ros-pkg-kdl/meshes/youbot_arm/arm1_convex.stl" />
 					<!--<cylinder length="0.102" radius="0.080"/>-->
 				</geometry>
@@ -92,5 +92,5 @@
 			<origin xyz="0 -0.032 0.078" rpy="0 0 0" />
 				<geometry>
-					<mesh filename="package://youbot_description/meshes/youbot_arm/arm2.dae" />
+					<mesh filename="package://youbot-ros-pkg-kdl/meshes/youbot_arm/arm2.dae" />
 				</geometry>
 				<material name="Orange" />
@@ -100,5 +100,5 @@
 				<origin xyz="0 -0.032 0.078" rpy="0 0 0" />
 				<geometry>
-					<mesh filename="package://youbot_description/meshes/youbot_arm/arm2_convex.stl" />
+					<mesh filename="package://youbot-ros-pkg-kdl/meshes/youbot_arm/arm2_convex.stl" />
 					<!--<box size="0.074 0.082 0.222"/>-->
 				</geometry>
@@ -126,5 +126,5 @@
 				<origin xyz="0.000 0.028 0.079" rpy="0 0 0" />
 				<geometry>
-					<mesh filename="package://youbot_description/meshes/youbot_arm/arm3.dae" />
+					<mesh filename="package://youbot-ros-pkg-kdl/meshes/youbot_arm/arm3.dae" />
 				</geometry>
 				<material name="Orange" />
@@ -134,5 +134,5 @@
 				<origin xyz="0.000 0.028 0.079" rpy="0 0 0" />
 				<geometry>
-					<mesh filename="package://youbot_description/meshes/youbot_arm/arm3_convex.stl" />
+					<mesh filename="package://youbot-ros-pkg-kdl/meshes/youbot_arm/arm3_convex.stl" />
 					<!--<box size="0.064 0.054 0.192"/>-->
 				</geometry>
@@ -160,5 +160,5 @@
 				<origin xyz="0 -0.010 0.029" rpy="0 0 0"/>
 				<geometry>
-					<mesh filename="package://youbot_description/meshes/youbot_arm/arm4.dae" />
+					<mesh filename="package://youbot-ros-pkg-kdl/meshes/youbot_arm/arm4.dae" />
 				</geometry>
 				<material name="Orange" />
@@ -168,5 +168,5 @@
 				<origin xyz="0 -0.010 0.029" rpy="0 0 0"/>
 				<geometry>
-					<mesh filename="package://youbot_description/meshes/youbot_arm/arm4_convex.stl" />
+					<mesh filename="package://youbot-ros-pkg-kdl/meshes/youbot_arm/arm4_convex.stl" />
 					<!--<box size="0.058 0.100 0.118"/>-->
 				</geometry>
@@ -193,5 +193,5 @@
 				<origin xyz="0.003 0 -0.034" rpy="0 0 0" />
 				<geometry>
-					<mesh filename="package://youbot_description/meshes/youbot_arm/arm5.dae" />
+					<mesh filename="package://youbot-ros-pkg-kdl/meshes/youbot_arm/arm5.dae" />
 				</geometry>
 				<material name="DarkGrey" />
@@ -200,5 +200,5 @@
 				<origin xyz="0.003 0 -0.034" rpy="0 0 0" />
 				<geometry>
-					<mesh filename="package://youbot_description/meshes/youbot_arm/arm5_convex.stl" />
+					<mesh filename="package://youbot-ros-pkg-kdl/meshes/youbot_arm/arm5_convex.stl" />
 					<!--<box size="0.054 0.096 0.030"/>-->
 				</geometry>

File: urdf/youbot_base/base.urdf.xacro (robot description, xacro)
@@ -5,7 +5,7 @@
         xmlns:xacro="http://ros.org/wiki/xacro">
 	<!-- sensors -->
-	<include filename="$(find youbot_description)/urdf/sensors/hokuyo_urg04_laser.urdf.xacro"/>
-	<include filename="$(find youbot_description)/urdf/youbot_base/base.gazebo.xacro" />
-	<include filename="$(find youbot_description)/urdf/youbot_base/base.transmission.xacro" />
+	<include filename="$(find youbot-ros-pkg-kdl)/urdf/sensors/hokuyo_urg04_laser.urdf.xacro"/>
+	<include filename="$(find youbot-ros-pkg-kdl)/urdf/youbot_base/base.gazebo.xacro" />
+	<include filename="$(find youbot-ros-pkg-kdl)/urdf/youbot_base/base.transmission.xacro" />
  	<!-- simplified box collision geometry for base -->
   	<property name="base_size_x" value="0.570" />
@@ -70,5 +70,5 @@
         			<origin xyz="0 0 0" rpy="0 0 0" />
         			<geometry>
-          				<mesh filename="package://youbot_description/meshes/youbot_base/base.dae"/>
+          				<mesh filename="package://youbot-ros-pkg-kdl/meshes/youbot_base/base.dae"/>
         			</geometry>
         			<material name="DarkGrey"/>
@@ -78,5 +78,5 @@
         			<geometry>
           				<!--<box size="${base_size_x} ${base_size_y} ${base_size_z}" />-->
-					<mesh filename="package://youbot_description/meshes/youbot_base/base_convex.stl"/>
+					<mesh filename="package://youbot-ros-pkg-kdl/meshes/youbot_base/base_convex.stl"/>
 	       			</geometry>
       			</collision>
@@ -122,5 +122,5 @@
       			<visual>
         			<origin xyz="0 0 0" rpy="0 0 0" />
-					<!--<mesh filename="package://youbot_description/meshes/youbot_base/youbot_wheel.stl" />-->
+					<!--<mesh filename="package://youbot-ros-pkg-kdl/meshes/youbot_base/youbot_wheel.stl" />-->
 				<geometry>
 					<sphere radius="${wheel_radius}"/>
@@ -172,5 +172,5 @@
         			<origin xyz="0 0 0" rpy="0 0 0" />
 				<geometry>
-          				<!--<mesh filename="package://youbot_description/meshes/youbot_base/youbot_wheel.stl" />-->
+          				<!--<mesh filename="package://youbot-ros-pkg-kdl/meshes/youbot_base/youbot_wheel.stl" />-->
 					<sphere radius="${wheel_radius}"/>
         			</geometry>
@@ -222,5 +222,5 @@
         			<origin xyz="0 0 0" rpy="0 0 0" />
 				<geometry>
-          				<!--<mesh filename="package://youbot_description/meshes/youbot_base/youbot_wheel.stl" />-->
+          				<!--<mesh filename="package://youbot-ros-pkg-kdl/meshes/youbot_base/youbot_wheel.stl" />-->
 					<sphere radius="${wheel_radius}"/>
         			</geometry>
@@ -271,5 +271,5 @@
         			<origin xyz="0 0 0" rpy="0 0 0" />
 				<geometry>
-          				<!--<mesh filename="package://youbot_description/meshes/youbot_base/youbot_wheel.stl" />-->
+          				<!--<mesh filename="package://youbot-ros-pkg-kdl/meshes/youbot_base/youbot_wheel.stl" />-->
 					<sphere radius="${wheel_radius}"/>
         			</geometry>

File: urdf/youbot_gripper/gripper.urdf.xacro (robot description, xacro)
@@ -4,7 +4,7 @@
        xmlns:interface="http://playerstage.sourceforge.net/gazebo/xmlschema/#interface"
        xmlns:xacro="http://ros.org/wiki/xacro">
-	<include filename="$(find youbot_description)/urdf/youbot_gripper/gripper.gazebo.xacro" />
-	<include filename="$(find youbot_description)/urdf/youbot_gripper/gripper.transmission.xacro" />
-	<include filename="$(find youbot_description)/urdf/youbot_gripper/limits.urdf.xacro" />
+	<include filename="$(find youbot-ros-pkg-kdl)/urdf/youbot_gripper/gripper.gazebo.xacro" />
+	<include filename="$(find youbot-ros-pkg-kdl)/urdf/youbot_gripper/gripper.transmission.xacro" />
+	<include filename="$(find youbot-ros-pkg-kdl)/urdf/youbot_gripper/limits.urdf.xacro" />
 	<xacro:macro name="youbot_gripper" params="parent name *origin">
 		<!-- joint between arm_7_link and sdh_palm_link -->
@@ -23,5 +23,5 @@
 				<origin xyz="0 0 0" rpy="0 0 0" />
 				<geometry>
-					<mesh filename="package://youbot_description/meshes/youbot_gripper/palm.stl" />
+					<mesh filename="package://youbot-ros-pkg-kdl/meshes/youbot_gripper/palm.stl" />
 				</geometry>
 				<material name="DarkGrey" />
@@ -31,5 +31,5 @@
 				<geometry>
 					<!--<box size="0.050 0.094 0.054"/>-->
-					<mesh filename="package://youbot_description/meshes/youbot_gripper/palm_convex.stl" />
+					<mesh filename="package://youbot-ros-pkg-kdl/meshes/youbot_gripper/palm_convex.stl" />
 				</geometry>
 			</collision>
@@ -53,5 +53,5 @@
 				<origin xyz="0 0 0" rpy="0 0 0" />
 				<geometry>
-					<mesh filename="package://youbot_description/meshes/youbot_gripper/finger.stl" />
+					<mesh filename="package://youbot-ros-pkg-kdl/meshes/youbot_gripper/finger.stl" />
 				</geometry>
 				<material name="DarkGrey" />
@@ -61,5 +61,5 @@
 				<geometry>
 					<!--<box size="0.014 0.020 0.046"/>-->
-					<mesh filename="package://youbot_description/meshes/youbot_gripper/finger_convex.stl" />
+					<mesh filename="package://youbot-ros-pkg-kdl/meshes/youbot_gripper/finger_convex.stl" />
 				</geometry>
 			</collision>
@@ -83,5 +83,5 @@
 				<origin xyz="0 0 0" rpy="0 0 0" />
 				<geometry>
-					<mesh filename="package://youbot_description/meshes/youbot_gripper/finger.stl" />
+					<mesh filename="package://youbot-ros-pkg-kdl/meshes/youbot_gripper/finger.stl" />
 				</geometry>
 				<material name="DarkGrey" />
@@ -91,5 +91,5 @@
 				<geometry>
 					<!--<box size="0.014 0.020 0.046"/>-->
-					<mesh filename="package://youbot_description/meshes/youbot_gripper/finger_convex.stl" />
+					<mesh filename="package://youbot-ros-pkg-kdl/meshes/youbot_gripper/finger_convex.stl" />
 				</geometry>
 			</collision>

File: urdf/youbot_plate/plate.urdf.xacro (robot description, xacro)
@@ -20,5 +20,5 @@
 				<origin xyz="0 0 0" rpy="0 0 0" />
 				<geometry>
-					<mesh filename="package://youbot_description/meshes/youbot_plate/plate.dae" />
+					<mesh filename="package://youbot-ros-pkg-kdl/meshes/youbot_plate/plate.dae" />
 				</geometry>
 				<material name="DarkGrey" />
@@ -27,5 +27,5 @@
 				<origin xyz="0 0 0" rpy="0 0 0" />
 				<geometry>
-					<mesh filename="package://youbot_description/meshes/youbot_plate/plate_convex.stl" />
+					<mesh filename="package://youbot-ros-pkg-kdl/meshes/youbot_plate/plate_convex.stl" />
 				</geometry>
 			</collision>
